Commit message: expanded env

File: src/my_robot_description/urdf/robot.urdf.xacro (robot description, xacro)
@@ -10,4 +10,11 @@
   <material name="black"><color rgba="0 0 0 1"/></material>
   <material name="gray"><color rgba="0.5 0.5 0.5 1"/></material>
+  <!-- Dummy World Link to Suppress KDL Warning -->
+  <link name="world"/>
+  <joint name="world_to_base" type="fixed">
+    <parent link="world"/>
+    <child link="base_link"/>
+    <origin xyz="0 0 0" rpy="0 0 0"/>
+  </joint>
   <!-- Base Link -->
   <link name="base_link">
@@ -25,5 +32,4 @@
       </geometry>
     </collision>
-    <!-- Inertia calculated as I_xx = m/12 * (width^2 + height^2), etc. for realistic physics -->
     <inertial>
       <mass value="5.0"/>
@@ -46,5 +52,4 @@
       </geometry>
     </collision>
-    <!-- Simple inertia for wheel -->
     <inertial>
       <mass value="0.5"/>
@@ -58,5 +63,5 @@
     <axis xyz="0 1 0"/>
   </joint>
-  <!-- Right Wheel (symmetric) -->
+  <!-- Right Wheel -->
   <link name="right_wheel_link">
     <visual>
@@ -73,5 +78,4 @@
       </geometry>
     </collision>
-    <!-- Simple inertia for wheel -->
     <inertial>
       <mass value="0.5"/>
@@ -100,14 +104,14 @@
       </geometry>
     </collision>
-    <!-- Simple inertia for caster -->
-    <inertial>
-      <mass value="0.2"/>
+    <inertial>
+      <mass value="0.5"/>
       <inertia ixx="0.0005" ixy="0" ixz="0" iyy="0.0005" iyz="0" izz="0.0005"/>
     </inertial>
   </link>
-  <joint name="caster_joint" type="fixed">
+  <joint name="caster_joint" type="continuous">
     <parent link="base_link"/>
     <child link="caster_wheel_link"/>
-    <origin xyz="${-chassis_length/2} 0 -${chassis_height/2}" rpy="0 0 0"/>
+    <origin xyz="${-chassis_length/2} 0 -${chassis_height}" rpy="0 0 0"/>
+    <axis xyz="0 0 1"/>
   </joint>
   <!-- IMU Link -->
@@ -126,5 +130,4 @@
       </geometry>
     </collision>
-    <!-- Negligible inertia for IMU -->
     <inertial>
       <mass value="0.01"/>
@@ -135,5 +138,5 @@
     <parent link="base_link"/>
     <child link="imu_link"/>
-    <origin xyz="0 0 0.05" rpy="0 0 0"/>
+    <origin xyz="0 0 ${chassis_height + 0.05}" rpy="0 0 0"/>
   </joint>
   <!-- LiDAR Link -->
@@ -152,5 +155,4 @@
       </geometry>
     </collision>
-    <!-- Simple inertia for LiDAR -->
     <inertial>
       <mass value="0.1"/>
@@ -161,5 +163,5 @@
     <parent link="base_link"/>
     <child link="lidar_link"/>
-    <origin xyz="0 0 0.2" rpy="0 0 0"/>
+    <origin xyz="0 0 ${chassis_height + 0.2}" rpy="0 0 0"/>
   </joint>
   <!-- Gazebo Plugins -->
@@ -169,14 +171,45 @@
     </plugin>
   </gazebo>
+  <!--
   <gazebo reference="base_link">
     <plugin filename="libgazebo_ros_diff_drive.so" name="diff_drive">
       <ros><namespace>/</namespace></ros>
-      <left_joint>left_wheel_joint</left_joint><right_joint>right_wheel_joint</right_joint>
-      <wheel_separation>${wheel_separation}</wheel_separation><wheel_diameter>${2 * wheel_radius}</wheel_diameter>
-      <max_wheel_torque>20</max_wheel_torque><max_wheel_acceleration>10</max_wheel_acceleration>
-      <publish_odom>true</publish_odom><odometry_topic>/gazebo_odom</odometry_topic>
-      <publish_wheel_tf>true</publish_wheel_tf><publish_wheel_joint_state>true</publish_wheel_joint_state>
+      <left_joint>left_wheel_joint</left_joint>
+      <right_joint>right_wheel_joint</right_joint>
+      <wheel_separation>${wheel_separation}</wheel_separation>
+      <wheel_diameter>${2 * wheel_radius}</wheel_diameter>
+      <max_wheel_torque>20</max_wheel_torque>
+      <max_wheel_acceleration>10</max_wheel_acceleration>
+      <publish_odom>true</publish_odom>
+      <odometry_topic>/gazebo_odom</odometry_topic>
+      <command_topic>/cmd_vel</command_topic>
+      <publish_wheel_tf>true</publish_wheel_tf>
+      <publish_wheel_joint_state>true</publish_wheel_joint_state>
+      <odometry_frame>odom</odometry_frame>
+      <robot_base_frame>base_link</robot_base_frame>
     </plugin>
   </gazebo>
+  -->
+  <gazebo>
+  <plugin name="diff_drive" filename="libgazebo_ros_diff_drive.so">
+    <ros>
+      <namespace>/</namespace>
+    </ros>
+    <left_joint>left_wheel_joint</left_joint>
+    <right_joint>right_wheel_joint</right_joint>
+    <wheel_separation>${wheel_separation}</wheel_separation>
+    <wheel_diameter>${2 * wheel_radius}</wheel_diameter>
+    <max_wheel_torque>20</max_wheel_torque>
+    <max_wheel_acceleration>10</max_wheel_acceleration>
+    <publish_odom>true</publish_odom>
+    <publish_odom_tf>true</publish_odom_tf>
+    <odometry_topic>gazebo_odom</odometry_topic>
+    <command_topic>cmd_vel</command_topic>
+    <publish_wheel_tf>true</publish_wheel_tf>
+    <publish_wheel_joint_state>true</publish_wheel_joint_state>
+    <odometry_frame>odom</odometry_frame>
+    <robot_base_frame>base_link</robot_base_frame>
+  </plugin>
+</gazebo>
   <gazebo reference="imu_link">
     <sensor name="imu_sensor" type="imu">
@@ -186,12 +219,9 @@
       <topic>/imu/data</topic>
       <plugin filename="libgazebo_ros_imu.so" name="imu_plugin">
-        <ros>
-          <namespace>/</namespace>
-          <remapping>~/out:=imu/data</remapping>
-        </ros>
+        <ros><namespace>/</namespace><remapping>~/out:=imu/data</remapping></ros>
         <gaussianNoise>0.0002</gaussianNoise>
         <orientation_covariance>0.0001 0 0 0 0.0001 0 0 0 0.0001</orientation_covariance>
-        <angular_velocity_covariance>0.0001 0 0 0 0.0001 0 0 0 0.0001</angular_velocity_covariance>
-        <linear_acceleration_covariance>0.0001 0 0 0 0.0001 0 0 0 0.0001</linear_acceleration_covariance>
+        <angular_velocity_covariance>0.0001 0 0 0 0 0.0001 0 0 0 0.0001</angular_velocity_covariance>
+        <linear_acceleration_covariance>0.0001 0 0 0 0 0.0001 0 0 0 0.0001</linear_acceleration_covariance>
       </plugin>
     </sensor>
@@ -219,8 +249,6 @@
       </ray>
       <plugin filename="libgazebo_ros_ray_sensor.so" name="lidar_plugin">
-        <ros>
-          <namespace>/</namespace>
-          <remapping>~/out:=scan</remapping>
-        </ros>
+        <ros><namespace>/</namespace><remapping>~/out:=scan</remapping></ros>
+        <output_type>sensor_msgs/LaserScan</output_type>
         <gaussianNoise>0.0001</gaussianNoise>
         <update_rate>10</update_rate>

Commit message: adding controller plugin -1

File: src/my_robot_description/urdf/robot.urdf.xacro (robot description, xacro)
@@ -167,6 +167,6 @@
   <!-- Gazebo Plugins -->
   <gazebo>
-    <plugin name="gazebo_ros_control" filename="libgazebo_ros_control.so">
-      <robotNamespace>/my_diffbot</robotNamespace>
+    <plugin name="gazebo_ros_control" filename="libgazebo_ros2_control.so">
+      <robotNamespace>my_diffbot</robotNamespace>
     </plugin>
   </gazebo>
@@ -190,5 +190,4 @@
     </plugin>
   </gazebo>
-  -->
   <gazebo>
   <plugin name="diff_drive" filename="libgazebo_ros_diff_drive.so">
@@ -212,4 +211,5 @@
   </plugin>
 </gazebo>
+-->
   <gazebo reference="imu_link">
     <sensor name="imu_sensor" type="imu">
@@ -218,5 +218,5 @@
       <visualize>true</visualize>
       <topic>/imu/data</topic>
-      <plugin filename="libgazebo_ros_imu.so" name="imu_plugin">
+      <plugin filename="libgazebo_ros_imu_sensor.so" name="imu_plugin">
         <ros><namespace>/</namespace><remapping>~/out:=imu/data</remapping></ros>
         <gaussianNoise>0.0002</gaussianNoise>
@@ -257,4 +257,5 @@
   </gazebo>
   <!-- Transmissions -->
+<!--
   <transmission name="left_wheel_trans">
     <type>transmission_interface/SimpleTransmission</type>
@@ -275,3 +276,43 @@
     </actuator>
   </transmission>
+-->
+  <transmission name="left_wheel_trans">
+  <type>transmission_interface/SimpleTransmission</type>
+  <joint name="left_wheel_joint">
+    <hardwareInterface>hardware_interface/VelocityJointInterface</hardwareInterface>
+  </joint>
+  <actuator name="left_wheel_motor">
+    <mechanicalReduction>1</mechanicalReduction>
+  </actuator>
+</transmission>
+<transmission name="right_wheel_trans">
+  <type>transmission_interface/SimpleTransmission</type>
+  <joint name="right_wheel_joint">
+    <hardwareInterface>hardware_interface/VelocityJointInterface</hardwareInterface>
+  </joint>
+  <actuator name="right_wheel_motor">
+    <mechanicalReduction>1</mechanicalReduction>
+  </actuator>
+</transmission>
+<ros2_control name="MyDiffBot" type="system">
+  <hardware>
+    <type>gazebo_ros2_control/GazeboSystem</type>  <!-- Foxy default Gazebo hardware plugin -->
+  </hardware>
+  <joint name="left_wheel_joint">
+    <command_interfaces>
+      <interface>velocity</interface>
+    </command_interfaces>
+    <state_interfaces>
+      <interface>velocity</interface>
+    </state_interfaces>
+  </joint>
+  <joint name="right_wheel_joint">
+    <command_interfaces>
+      <interface>velocity</interface>
+    </command_interfaces>
+    <state_interfaces>
+      <interface>velocity</interface>
+    </state_interfaces>
+  </joint>
+</ros2_control>
 </robot>

Commit message: ros2 control - 3

File: src/my_robot_description/urdf/robot.urdf.xacro (robot description, xacro)
@@ -51,4 +51,12 @@
         <cylinder radius="${wheel_radius}" length="0.05"/>
       </geometry>
+      <surface>
+        <friction>
+          <ode>
+            <mu>1.0</mu>
+            <mu2>1.0</mu2>
+          </ode>
+        </friction>
+      </surface>
     </collision>
     <inertial>
@@ -77,4 +85,12 @@
         <cylinder radius="${wheel_radius}" length="0.05"/>
       </geometry>
+      <surface>
+        <friction>
+          <ode>
+            <mu>1.0</mu>
+            <mu2>1.0</mu2>
+          </ode>
+        </friction>
+      </surface>
     </collision>
     <inertial>
@@ -166,50 +182,4 @@
   </joint>
   <!-- Gazebo Plugins -->
-  <gazebo>
-    <plugin name="gazebo_ros_control" filename="libgazebo_ros2_control.so">
-      <robotNamespace>my_diffbot</robotNamespace>
-    </plugin>
-  </gazebo>
-  <!--
-  <gazebo reference="base_link">
-    <plugin filename="libgazebo_ros_diff_drive.so" name="diff_drive">
-      <ros><namespace>/</namespace></ros>
-      <left_joint>left_wheel_joint</left_joint>
-      <right_joint>right_wheel_joint</right_joint>
-      <wheel_separation>${wheel_separation}</wheel_separation>
-      <wheel_diameter>${2 * wheel_radius}</wheel_diameter>
-      <max_wheel_torque>20</max_wheel_torque>
-      <max_wheel_acceleration>10</max_wheel_acceleration>
-      <publish_odom>true</publish_odom>
-      <odometry_topic>/gazebo_odom</odometry_topic>
-      <command_topic>/cmd_vel</command_topic>
-      <publish_wheel_tf>true</publish_wheel_tf>
-      <publish_wheel_joint_state>true</publish_wheel_joint_state>
-      <odometry_frame>odom</odometry_frame>
-      <robot_base_frame>base_link</robot_base_frame>
-    </plugin>
-  </gazebo>
-  <gazebo>
-  <plugin name="diff_drive" filename="libgazebo_ros_diff_drive.so">
-    <ros>
-      <namespace>/</namespace>
-    </ros>
-    <left_joint>left_wheel_joint</left_joint>
-    <right_joint>right_wheel_joint</right_joint>
-    <wheel_separation>${wheel_separation}</wheel_separation>
-    <wheel_diameter>${2 * wheel_radius}</wheel_diameter>
-    <max_wheel_torque>20</max_wheel_torque>
-    <max_wheel_acceleration>10</max_wheel_acceleration>
-    <publish_odom>true</publish_odom>
-    <publish_odom_tf>true</publish_odom_tf>
-    <odometry_topic>gazebo_odom</odometry_topic>
-    <command_topic>cmd_vel</command_topic>
-    <publish_wheel_tf>true</publish_wheel_tf>
-    <publish_wheel_joint_state>true</publish_wheel_joint_state>
-    <odometry_frame>odom</odometry_frame>
-    <robot_base_frame>base_link</robot_base_frame>
-  </plugin>
-</gazebo>
--->
   <gazebo reference="imu_link">
     <sensor name="imu_sensor" type="imu">
@@ -256,63 +226,29 @@
     </sensor>
   </gazebo>
-  <!-- Transmissions -->
-<!--
-  <transmission name="left_wheel_trans">
-    <type>transmission_interface/SimpleTransmission</type>
-    <joint name="left_wheel_joint">
-      <hardwareInterface>hardware_interface/PositionJointInterface</hardwareInterface>
-    </joint>
-    <actuator name="left_wheel_motor">
-      <mechanicalReduction>1</mechanicalReduction>
-    </actuator>
-  </transmission>
-  <transmission name="right_wheel_trans">
-    <type>transmission_interface/SimpleTransmission</type>
-    <joint name="right_wheel_joint">
-      <hardwareInterface>hardware_interface/PositionJointInterface</hardwareInterface>
-    </joint>
-    <actuator name="right_wheel_motor">
-      <mechanicalReduction>1</mechanicalReduction>
-    </actuator>
-  </transmission>
--->
-  <transmission name="left_wheel_trans">
-  <type>transmission_interface/SimpleTransmission</type>
-  <joint name="left_wheel_joint">
-    <hardwareInterface>hardware_interface/VelocityJointInterface</hardwareInterface>
-  </joint>
-  <actuator name="left_wheel_motor">
-    <mechanicalReduction>1</mechanicalReduction>
-  </actuator>
-</transmission>
-<transmission name="right_wheel_trans">
-  <type>transmission_interface/SimpleTransmission</type>
-  <joint name="right_wheel_joint">
-    <hardwareInterface>hardware_interface/VelocityJointInterface</hardwareInterface>
-  </joint>
-  <actuator name="right_wheel_motor">
-    <mechanicalReduction>1</mechanicalReduction>
-  </actuator>
-</transmission>
-<ros2_control name="MyDiffBot" type="system">
-  <hardware>
-    <type>gazebo_ros2_control/GazeboSystem</type>  <!-- Foxy default Gazebo hardware plugin -->
-  </hardware>
-  <joint name="left_wheel_joint">
-    <command_interfaces>
-      <interface>velocity</interface>
-    </command_interfaces>
-    <state_interfaces>
-      <interface>velocity</interface>
-    </state_interfaces>
-  </joint>
-  <joint name="right_wheel_joint">
-    <command_interfaces>
-      <interface>velocity</interface>
-    </command_interfaces>
-    <state_interfaces>
-      <interface>velocity</interface>
-    </state_interfaces>
-  </joint>
-</ros2_control>
+  <ros2_control name="GazeboSystem" type="system">
+        <hardware>
+            <plugin>gazebo_ros2_control/GazeboSystem</plugin>
+        </hardware>
+        <joint name="left_wheel_joint">
+            <command_interface name="velocity">
+                <param name="min">-10</param>
+                <param name="max">10</param>
+            </command_interface>
+            <state_interface name="velocity"/>
+            <state_interface name="position"/>
+        </joint>
+        <joint name="right_wheel_joint">
+            <command_interface name="velocity">
+                <param name="min">-10</param>
+                <param name="max">10</param>
+            </command_interface>
+            <state_interface name="velocity"/>
+            <state_interface name="position"/>
+        </joint>
+    </ros2_control>
+    <gazebo>
+        <plugin name="gazebo_ros2_control" filename="libgazebo_ros2_control.so">
+            <parameters>$(find my_simulation)/config/diffbot_controllers.yaml</parameters>
+        </plugin>
+    </gazebo>
 </robot>

Commit message: ros2_control - working

File: src/my_robot_description/urdf/robot.urdf.xacro (robot description, xacro)
@@ -10,11 +10,4 @@
   <material name="black"><color rgba="0 0 0 1"/></material>
   <material name="gray"><color rgba="0.5 0.5 0.5 1"/></material>
-  <!-- Dummy World Link to Suppress KDL Warning -->
-  <link name="world"/>
-  <joint name="world_to_base" type="fixed">
-    <parent link="world"/>
-    <child link="base_link"/>
-    <origin xyz="0 0 0" rpy="0 0 0"/>
-  </joint>
   <!-- Base Link -->
   <link name="base_link">

Commit message: fix rotation of wheels

File: src/my_robot_description/urdf/robot.urdf.xacro (robot description, xacro)
@@ -33,5 +33,5 @@
   <link name="left_wheel_link">
     <visual>
-      <origin xyz="0 0 0" rpy="0 0 0"/>
+      <origin xyz="0 0 0" rpy="0 1.5707 1.5707"/>
       <geometry>
         <cylinder radius="${wheel_radius}" length="0.05"/>
@@ -40,5 +40,5 @@
     </visual>
     <collision>
-      <origin xyz="0 0 0" rpy="0 0 0"/>
+      <origin xyz="0 0 0" rpy="0 1.5707 1.5707"/>
       <geometry>
         <cylinder radius="${wheel_radius}" length="0.05"/>
@@ -61,5 +61,5 @@
     <parent link="base_link"/>
     <child link="left_wheel_link"/>
-    <origin xyz="${chassis_length/2} ${-wheel_separation/2} 0" rpy="1.5708 0 0"/>
+    <origin xyz="${chassis_length/2} ${-wheel_separation/2} 0" rpy="0 0 0"/>
     <axis xyz="0 1 0"/>
   </joint>
@@ -67,5 +67,5 @@
   <link name="right_wheel_link">
     <visual>
-      <origin xyz="0 0 0" rpy="0 0 0"/>
+      <origin xyz="0 0 0" rpy="0 1.5707 1.5707"/>
       <geometry>
         <cylinder radius="${wheel_radius}" length="0.05"/>
@@ -74,5 +74,5 @@
     </visual>
     <collision>
-      <origin xyz="0 0 0" rpy="0 0 0"/>
+      <origin xyz="0 0 0" rpy="0 1.5707 1.5707"/>
       <geometry>
         <cylinder radius="${wheel_radius}" length="0.05"/>
@@ -95,33 +95,34 @@
     <parent link="base_link"/>
     <child link="right_wheel_link"/>
-    <origin xyz="${chassis_length/2} ${wheel_separation/2} 0" rpy="1.5708 0 0"/>
+    <origin xyz="${chassis_length/2} ${wheel_separation/2} 0" rpy="0 0 0"/>
     <axis xyz="0 1 0"/>
   </joint>
-  <!-- Caster -->
-  <link name="caster_wheel_link">
-    <visual>
-      <origin xyz="0 0 0" rpy="0 0 0"/>
-      <geometry>
-        <sphere radius="0.025"/>
-      </geometry>
-      <material name="gray"/>
-    </visual>
-    <collision>
-      <origin xyz="0 0 0" rpy="0 0 0"/>
-      <geometry>
-        <sphere radius="0.025"/>
-      </geometry>
-    </collision>
-    <inertial>
-      <mass value="0.5"/>
-      <inertia ixx="0.0005" ixy="0" ixz="0" iyy="0.0005" iyz="0" izz="0.0005"/>
-    </inertial>
-  </link>
-  <joint name="caster_joint" type="continuous">
-    <parent link="base_link"/>
-    <child link="caster_wheel_link"/>
-    <origin xyz="${-chassis_length/2} 0 -${chassis_height}" rpy="0 0 0"/>
-    <axis xyz="0 0 1"/>
-  </joint>
+   <!-- Caster Wheel -->
+<link name="caster_wheel_link">
+  <visual>
+    <origin xyz="0 0 0" rpy="0 0 0"/>
+    <geometry>
+      <sphere radius="0.025"/>
+    </geometry>
+    <material name="gray"/>
+  </visual>
+  <collision>
+    <origin xyz="0 0 0" rpy="0 0 0"/>
+    <geometry>
+      <sphere radius="0.025"/>
+    </geometry>
+  </collision>
+  <inertial>
+    <mass value="0.2"/>
+    <!-- Solid sphere inertia - I = 2/5 * m * r^2 -->
+    <inertia ixx="0.00005" ixy="0" ixz="0"
+	     iyy="0.00005" iyz="0" izz="0.00005"/>
+  </inertial>
+</link>
+<joint name="caster_joint" type="continuous">
+  <parent link="base_link"/>
+  <child link="caster_wheel_link"/>
+  <origin xyz="${-chassis_length/2 + 0.05} 0 -${wheel_radius}" rpy="0 0 0"/>
+</joint>
   <!-- IMU Link -->
   <link name="imu_link">
